Commit message: Update my_robot.xacro

File: my_robot/urdf/my_robot.xacro (robot description, xacro)
@@ -48,6 +48,6 @@
     </visual>
   </link>
-  <!--Link (right_wheel)-->
-  <link name='right_wheel'>
+  <!--Link (left_wheel)-->
+  <link name='left_wheel'>
     <inertial>
       <mass value="5"/>
@@ -59,12 +59,12 @@
       />
     </inertial>
-    <collision name='right_wheel_collision'>
-      <origin rpy="0 1.5707 1.5707" xyz="0 0 0" />
+    <collision name='left_wheel_collision'>
+      <origin  xyz="0 0 0" rpy="0 1.5707 1.5707"/>
       <geometry>
         <cylinder length="0.05" radius="0.1"/>
       </geometry>
     </collision>
-    <visual name='right_wheel_visual'>
-      <origin rpy="0 1.5707 1.5707" xyz="0 0 0"/>
+    <visual name='left_wheel_visual'>
+      <origin xyz="0 0 0" rpy="0 1.5707 1.5707"/>
       <geometry>
         <cylinder length="0.05" radius="0.1"/>
@@ -72,8 +72,8 @@
     </visual>
   </link>
-  <!--Joint (right_wheel_hinge)-->
-  <joint name="right_wheel_hinge" type="continuous">
+  <!--Joint (left_wheel_hinge)-->
+  <joint name="left_wheel_hinge" type="continuous">
     <origin xyz="-0.05 0.15 0" rpy="0 0 0"/>
-    <child link="right_wheel" />
+    <child link="left_wheel" />
     <parent link="chassis"/>
     <axis xyz="0 1 0" rpy="0 0 0" />
@@ -81,6 +81,6 @@
     <joint_properties damping="1.0" friction="1.0" />
   </joint>
-  <!--Link (left_wheel)-->
-  <link name="left_wheel">
+  <!--Link (right_wheel)-->
+  <link name="right_wheel">
     <inertial>
       <origin xyz="0 0 0" rpy="0 1.5707 1.5707" />
@@ -92,5 +92,5 @@
       />
     </inertial>
-    <collision name="left_wheel_collision">
+    <collision name="right_wheel_collision">
       <origin xyz="0 0 0" rpy="0 1.5707 1.5707"/>
       <geometry>
@@ -98,6 +98,6 @@
       </geometry>
     </collision>
-    <visual name="left_wheel_visual">
-      <origin rpy="0 1.5707 1.5707" xyz="0 0 0"/>
+    <visual name="right_wheel_visual">
+      <origin xyz="0 0 0" rpy="0 1.5707 1.5707"/>
       <geometry>
         <cylinder length="0.05" radius="0.1"/>
@@ -105,8 +105,8 @@
     </visual>
   </link>
-  <!--Joint (left_wheel_hinge)-->
-  <joint name="left_wheel_hinge" type="continuous">
+  <!--Joint (right_wheel_hinge)-->
+  <joint name="right_wheel_hinge" type="continuous">
     <origin xyz="-0.05 -0.15 0" rpy="0 0 0"/>
-    <child link="left_wheel" />
+    <child link="right_wheel" />
     <parent link="chassis"/>
     <axis rpy="0 0 0" xyz="0 1 0"/>
